Commit message: fixing some axis directions in urdf

File: data/panda_hand2.urdf (robot description, URDF)
Before this commit: robot panda, 7 links, 6 joints
Joints:
- joint panda_hand_xbase: axis 0 0 1 -> 0 1 0
- joint panda_left_fingerpad_joint: axis 0 0 1 -> (none)
- joint panda_right_fingerpad_joint: axis 0 0 1 -> (none)

Commit message: added visualizations of forces. Separated FT sensor into its own object. Added utils sleeper

File: data/panda_hand2.urdf (robot description, URDF)
Before this commit: robot panda, 7 links, 6 joints
Links:
- added link panda_wbase
- added link panda_ybase
- link panda_leftfinger: mass 0.1 -> 0.026
- link panda_leftfingerpad: mass 0.003 -> 0.0000000000003
- link panda_rightfinger: mass 0.1 -> 0.026
- link panda_rightfingerpad: mass 0.003 -> 0.0000000000003
- link panda_xbase: mass .5 -> None; geometry 
Joints:
- added joint panda_hand_wbase: type revolute, parent panda_wbase, child panda_hand, origin xyz=0. 0. 0. rpy=0 0 0, axis 1 0 0, limit effort=10 velocity=0.02
- added joint panda_hand_ybase: type prismatic, parent panda_ybase, child panda_wbase, origin xyz=0. 0. 0. rpy=0 0 0, axis 0 0 1, limit effort=10 velocity=0.1
- joint panda_finger_left: axis 0 1 0 -> 0 -1 0
- joint panda_finger_right: axis 0 -1 0 -> 0 1 0
- joint panda_hand_xbase: child panda_hand -> panda_ybase; limit lower=-0.2 upper=0.2 effort=1000 velocity=5.0 -> effort=10 velocity=0.1; origin xyz=0.05 0. 0. rpy=1.57079632679 0 1.57079632679 -> xyz=0. 0. 0. rpy=1.57079632679 0 1.57079632679
- joint panda_xbase_zbase: origin xyz=0.05 0 0.1 rpy=1.57079632679 0 0 -> xyz=0.1 0 0.1 rpy=1.57079632679 0 0

Commit message: added sensor object to frankaHand and got compliance control to work.

File: data/panda_hand2.urdf (robot description, URDF)
Before this commit: robot panda, 9 links, 8 joints
Links:
- link panda_hand: mass .81 -> .0081
- link panda_wbase: mass None -> .001
- link panda_xbase: mass None -> .001
- link panda_ybase: mass None -> .001

Commit message: fixed the hand urdf so that the frames show up in the right place. Also, changed the mug sdf to be more fine grained. Changed the control for compliant contact to use only 3 DOF and inverse Jacobian.

File: data/panda_hand2.urdf (robot description, URDF)
Before this commit: robot panda, 9 links, 8 joints
Links:
- link panda_rightfinger: geometry 
- link panda_rightfingerpad: geometry 
Joints:
- joint panda_left_fingerpad_joint: origin xyz=0 0 0.045 rpy=0 0 0 -> xyz=0 -0.009 0.045 rpy=0 0 0
- joint panda_right_fingerpad_joint: origin xyz=0 0 0.045 rpy=0 0 0 -> xyz=0 0.009 0.045 rpy=0 0 3.14159265359
